File: pcb/KnowledgeBoard.kicad_pcb (KiCad board)
At the start: 2 copper layers, 61.5 x 81 mm, 32 parts, among them SW1 RotaryEncoder_Switch, SW10 SW_Push, SW11 SW_Push, SW2 RotaryEncoder_Switch, SW3 SW_Push, SW4 SW_Push, SW5 SW_Push, SW6 SW_Push, SW7 SW_Push, SW8 SW_Push, SW9 SW_Push, U1 MOUDLE-SEEEDUINO-XIAO

Commit message: Pre-flight ready
Parts:
- D1, D12, D13, D14, D2, D3, D6, D7, D8: footprint CustomLibrary:SK6812MINI-E_Fixed -> footprints:SK6812MINI-E_fixed
Routing:
- net Col1: track 72.6 -> 70.9 mm
Other:
- outline, holes or cut-outs redrawn
- board text added: "KnowledgeBoard V1"
