File: pcb/KnowledgeBoard.kicad_sch (KiCad schematic)
At the start: 32 parts, among them SW1 RotaryEncoder_Switch, SW10 SW_Push, SW11 SW_Push, SW2 RotaryEncoder_Switch, SW3 SW_Push, SW4 SW_Push, SW5 SW_Push, SW6 SW_Push, SW7 SW_Push, SW8 SW_Push, SW9 SW_Push, U1 MOUDLE-SEEEDUINO-XIAO

Commit message: Pre-flight ready
Parts:
- D1, D12, D13, D14, D2, D3, D6, D7, D8: footprint CustomLibrary:SK6812MINI-E_Fixed -> footprints:SK6812MINI-E_fixed
Other:
- moved on the sheet: D4, D5
